File: electronics/MovingTargetUnit/v1/MovingTargetUnit_v4.sch (EAGLE design)
At the start: 37 parts, among them J1 PINHDR_1X6-JST, J2 PINHDR_1X6-JST, J3 PINHDR_1X3XH-JST, J4 PINHDR_1X3XH-JST, J5 PINHDR_1X3XH-JST, J6 PINHDR_1X4-JST, J7 PINHDR_1X6-JST, M1 ESP8266_MODULE, P1 10K, U1 LM2902, U2 VREG-3L7805CDT, U3 VREG-3L7805CDT, U4 74ABT125-D

Commit message: FIxing Doc, Fixing Intellasense, New Schematics
Other:
- note added: "MOVING TARGET UNIT, V4"
- note removed: "MOVING TARGET UNIT"
Changed lines of the file:
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@@
 <plain>
 <text x="111.252" y="103.124" size="1.4224" layer="97">TO NEO 1</text>
-<text x="48.26" y="116.84" size="5.08" layer="97">MOVING TARGET UNIT</text>
+<text x="48.26" y="116.84" size="5.08" layer="97">MOVING TARGET UNIT, V4</text>
 <text x="111.506" y="86.106" size="1.4224" layer="97">TO NEO 2</text>
 <text x="60.96" y="5.08" size="1.6764" layer="97">2S Lipo Bat
